File: Row-of-4-pots/Row-of-4-pots.kicad_sch (KiCad schematic)
At the start: 10 parts, among them J1 Conn_02x03_Odd_Even, J2 Conn_02x03_Odd_Even, J3 RV, J4 PWR, J5 PWR, J6 RV

Commit message: Final version 1.0 ordered
Parts:
- J1, J2: value Conn_02x03_Odd_Even -> FHMD-DA006G1NBON-B
- J3, J6: value RV -> S3B-XH-A; footprint Connector_PinHeader_2.54mm:PinHeader_1x03_P2.54mm_Horizontal -> Connector_JST:JST_XH_S3B-XH-A_1x03_P2.50mm_Horizontal
- J4, J5: value PWR -> S3B-XH-A; footprint Connector_PinHeader_2.54mm:PinHeader_1x03_P2.54mm_Horizontal -> Connector_JST:JST_XH_S3B-XH-A_1x03_P2.50mm_Horizontal
Other:
- title: (none) -> Row-of-4-POTs
Changed lines of the file:
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@@
 	(generator_version "8.0")
 	(paper "A4")
+	(title_block
+		(title "Row-of-4-POTs")
+		(date "2024-11-23")
+		(rev "1.0")
+	)
 	(junction
 		(at 177.8 91.44)
@@
 			)
 		)
-		(property "Value" "RV"
+		(property "Value" "S3B-XH-A"
 			(at 195.072 78.5637 0)
 			(effects
@@
 			)
 		)
-		(property "Footprint" "Connector_PinHeader_2.54mm:PinHeader_1x03_P2.54mm_Horizontal"
+		(property "Footprint" "Connector_JST:JST_XH_S3B-XH-A_1x03_P2.50mm_Horizontal"
 			(at 196.85 83.82 0)
 			(effects
@@
 			)
 		)
-		(property "Datasheet" "~"
+		(property "Datasheet" "455-S3B-XH-A-ND"
 			(at 196.85 83.82 0)
 			(effects
@@
 			)
 		)
-		(property "Value" "PWR"
+		(property "Value" "S3B-XH-A"
 			(at 52.578 96.3437 0)
 			(effects
@@
 			)
 		)
-		(property "Footprint" "Connector_PinHeader_2.54mm:PinHeader_1x03_P2.54mm_Horizontal"
+		(property "Footprint" "Connector_JST:JST_XH_S3B-XH-A_1x03_P2.50mm_Horizontal"
 			(at 50.8 101.6 0)
 			(effects
@@
 			)
 		)
-		(property "Datasheet" "~"
+		(property "Datasheet" "455-S3B-XH-A-ND"
 			(at 50.8 101.6 0)
 			(effects
@@
 			)
 		)
-		(property "Value" "Conn_02x03_Odd_Even"
+		(property "Value" "FHMD-DA006G1NBON-B"
 			(at 168.91 105.0782 0)
 			(effects
@@
 			)
 		)
-		(property "Datasheet" "~"
+		(property "Datasheet" "4324-FHMD-DA006G1NBON-B-ND"
 			(at 167.64 110.49 0)
 			(effects
@@
 			)
 		)
-		(property "Value" "PWR"
+		(property "Value" "S3B-XH-A"
 			(at 52.578 78.5637 0)
 			(effects
@@
 			)
 		)
-		(property "Footprint" "Connector_PinHeader_2.54mm:PinHeader_1x03_P2.54mm_Horizontal"
+		(property "Footprint" "Connector_JST:JST_XH_S3B-XH-A_1x03_P2.50mm_Horizontal"
 			(at 50.8 83.82 0)
 			(effects
@@
 			)
 		)
-		(property "Datasheet" "~"
+		(property "Datasheet" "455-S3B-XH-A-ND"
 			(at 50.8 83.82 0)
 			(effects
@@
 			)
 		)
-		(property "Description" "Potentiometer, US symbol"
+		(property "Description" "RD901F-40-15K-B10K"
 			(at 90.17 83.82 0)
 			(effects
@@
 			)
 		)
-		(property "Value" "RV"
+		(property "Value" "S3B-XH-A"
 			(at 195.072 91.2637 0)
 			(effects
@@
 			)
 		)
-		(property "Footprint" "Connector_PinHeader_2.54mm:PinHeader_1x03_P2.54mm_Horizontal"
+		(property "Footprint" "Connector_JST:JST_XH_S3B-XH-A_1x03_P2.50mm_Horizontal"
 			(at 196.85 96.52 0)
 			(effects
@@
 			)
 		)
-		(property "Datasheet" "~"
+		(property "Datasheet" "455-S3B-XH-A-ND"
 			(at 196.85 96.52 0)
 			(effects
@@
 			)
 		)
-		(property "Value" "Conn_02x03_Odd_Even"
+		(property "Value" "FHMD-DA006G1NBON-B"
 			(at 125.73 122.8582 0)
 			(effects
@@
 			)
 		)
-		(property "Datasheet" "~"
+		(property "Datasheet" "4324-FHMD-DA006G1NBON-B-ND"
 			(at 124.46 128.27 0)
 			(effects
