File: Row-of-4-pots/Row-of-4-pots.kicad_pcb (KiCad board)
At the start: 4 copper layers, 91.4 x 19 mm, 10 parts, among them J1 Conn_02x03_Odd_Even, J2 Conn_02x03_Odd_Even, J3 RV, J4 PWR, J5 PWR, J6 RV

Commit message: Final version 1.0 ordered
Parts:
- J3: value RV -> S3B-XH-A; footprint Connector_PinHeader_2.54mm:PinHeader_1x03_P2.54mm_Horizontal -> Connector_JST:JST_XH_S3B-XH-A_1x03_P2.50mm_Horizontal
- J4: value PWR -> S3B-XH-A; footprint Connector_PinHeader_2.54mm:PinHeader_1x03_P2.54mm_Horizontal -> Connector_JST:JST_XH_S3B-XH-A_1x03_P2.50mm_Horizontal; moved to B.Cu
- J5: value PWR -> S3B-XH-A; footprint Connector_PinHeader_2.54mm:PinHeader_1x03_P2.54mm_Horizontal -> Connector_JST:JST_XH_S3B-XH-A_1x03_P2.50mm_Horizontal; moved to F.Cu
- J6: value RV -> S3B-XH-A; footprint Connector_PinHeader_2.54mm:PinHeader_1x03_P2.54mm_Horizontal -> Connector_JST:JST_XH_S3B-XH-A_1x03_P2.50mm_Horizontal; moved to F.Cu
- moved RV1 76.2 mm to (213.3, 99.1)
- moved RV4 76.2 mm to (137.1, 99.1)
- moved J3 64.0 mm to (144.8, 94.0), turned to 0 degrees
- moved J1 50.8 mm to (200.7, 88.3)
- moved J2 50.8 mm to (149.9, 88.3)
- moved RV2 25.4 mm to (187.9, 99.1)
- moved RV3 25.4 mm to (162.5, 99.1)
- moved J5 5.08 mm to (170.2, 94.0), turned to 0 degrees
- moved J6 5.08 mm to (195.6, 94.0), turned to 0 degrees
- moved J4 3.81 mm to (170.2, 92.1), turned to 0 degrees
Routing:
- net /VCC/2: track 65.9 -> 0.00 mm
- net /P1: track 108.2 -> 87.2 mm
- net /P2: track 95.5 -> 86.8 mm
- net /R3: track 20.5 -> 15.4 mm
- net /R1: track 19.9 -> 15.4 mm
- net /R4: track 19.7 -> 15.9 mm
- net /R2: track 19.7 -> 16.2 mm
- net VCC: track 64.8 -> 64.2 mm
- added copper zone on In2.Cu, net /VCC/2
- removed copper zone on In2.Cu, net GNDA
Other:
- board text added: "Front"
- board text added: "JM: Row-of-4-pots, v1.0, 2024/11/23"
- board text added: "RV3"
- board text added: "RV4"
- board text added: "VCC/2"
- board text removed: "<-GND->"
- board text removed: "<-VC2->"
- board text removed: "<-VCC->"
- board text removed: "JM: Row-of-4-pots, v1.0, 2024/11"
