File: 2-Band-EQ-Board/2-Band-EQ-Board.kicad_pcb (KiCad board)
At the start: 4 copper layers, 29.2 x 22.9 mm, 18 parts, among them J1 Conn_02x03_Odd_Even, U1 TL072

Commit message: Final version 1.0 ordered
Parts:
- C1: value 100n -> 33n
- C11, C9: value 3.3u -> 1.5u
- C2: value 3.3u -> 0.68u
- C3: value 56n -> 15n
- C4: value 1.5u -> 0.33u
- J1: value Conn_02x03_Odd_Even -> PHED-DS006G1ABOGA-A006
- U1: value TL072 -> 296-TL072HIDRCT-ND
Other:
- board text added: "JM: 2-Band-Gyrator, v1.0, 2024/11/23"
- board text removed: "JM: 2-Band-EQ-Board, v1.0, 2024/11"
- board text removed: "VCC/2"
